File: pcb/syncbox.kicad_pcb (KiCad board)
At the start: 2 copper layers, 158 x 34 mm, 100 parts, among them J1 DC 7-12V, J2 SWD, J3 USB_B, J4 IN, J5 SYNC1, J6 SYNC2, J7 Gate 1, J8 Gate 2, J9 Gate 3, Q1 PMBT2907A, Q2 PMBT2907A, Q3 PMBT2907A, Q4 PMBT2907A, Q5 PMBT2907A, Q6 PMBT2907A, Q7 PMBT2907A, Q8 PMBT2907A, Q9 PMBT2907A, U1 LD1117S50TR_SOT223, U2 STM32F303RET6, U3 ADP150, U4 RV1S9160A, U5 CD74HCT04, X1 ECS-TXO-2520 24MHz

Commit message: Version 1.1 hardware changes
Parts:
- removed TP1: E5V, Syncbox:TestPoint_Pad_D1.5mm
- removed TP6: U5V, Syncbox:TestPoint_Pad_D1.5mm
- added Q10: MMBT2222A, Package_TO_SOT_SMD:SOT-23_Handsoldering, F.Cu at (101.3, 80.9)
- added R33: 10k, Resistor_SMD:R_0805_2012Metric_Pad1.20x1.40mm_HandSolder, F.Cu at (101.3, 87.2)
- added R34: 100, Resistor_SMD:R_0805_2012Metric_Pad1.20x1.40mm_HandSolder, F.Cu at (96.4, 81.7)
- added R35: 36k, Resistor_SMD:R_0805_2012Metric_Pad1.20x1.40mm_HandSolder, F.Cu at (101.3, 85.2)
- D2, D6, D7: value BAT42 -> BAT60J; footprint Syncbox:D_0805_2012Metric_Pad1.15x1.40mm_HandSolder -> Diode_SMD:D_SOD-323_HandSoldering
- D3, D4, D5: value TVS -> TVS PGB1010603
- JP1: value DFU -> B0
- R2: value 1k5 -> 1.5k
- moved C4 2.50 mm to (85.8, 82.0)
- moved C8 2.45 mm to (101.3, 89.2)
- moved R2 2.03 mm to (90.5, 82.0)
- moved C7 1.40 mm to (101.3, 91.2)
- moved C10 0.75 mm to (104.5, 83.5), turned to 0 degrees
Connections:
- net Net-(C10-Pad1) renamed U5V
- net Net-(C2-Pad1) renamed /E5V
- R2 pad 1: USBD_P -> Net-(Q10-Pad2)
- R2 pad 2: +3V3 -> USBD_P
- U2 pad 42: unconnected-(U2-Pad42) -> SENSE
Routing:
- net Net-(Q10-Pad1): track 0.00 -> 14.5 mm
- net Net-(Q10-Pad2): track 0.00 -> 9.90 mm
- net SENSE: track 0.00 -> 6.68 mm
- net +3V3: track 77.6 -> 83.9 mm
- net U5V: track 10.7 -> 16.9 mm
- net USBD_N: track 8.52 -> 9.15 mm
- net GND: vias 39 -> 40
Other:
- board text added: "syncbox v1.1"
- board text removed: "E5V"
- board text removed: "U5V"
- board text removed: "syncbox v1.0"
